File: atari_punk.kicad_pcb (KiCad board)
At the start: 2 copper layers, 52.7 x 45.1 mm, 16 parts, among them J1 Conn_01x02_Male, J2 Conn_01x02_Male, SW1 SK12D07VG4, U1 NE555P, U2 NE555P

Commit message: Se agrandan los pad de chasis de los potenciómetros.
Parts:
- R1, R4: footprint Potentiometer_THT:Potentiometer_Alpha_RD901F-40-00D_Single_Vertical -> eduardofilo_footprints:Potentiometer_Alpha_RD901F-40-00D_Single_Vertical_mod
