File: atari_punk.kicad_pcb (KiCad board)
At the start: 2 copper layers, 52.7 x 45.1 mm, 16 parts, among them J1 Conn_01x02_Male, J2 Conn_01x02_Male, SW1 SK12D07VG4, U1 NE555P, U2 NE555P

Commit message: v6 en silkscreen.
Other:
- board text added: "Atari Punk v6"
- board text removed: "Atari Punk v5"
